File: _autosave-DDR.sch (KiCad schematic (older format))
At the start: 37 parts, among them U1 IMX6UL_BGA289, U2 DDR3_BGA96

Commit message: Completed DDR routing & length matching
Parts:
- removed C43: 4.7uF, Capacitor_SMD:C_0402_1005Metric, symbol Device:CP1
Connections:
- wire segments 301 -> 297
Changed lines of the file:
@@
-$Comp
-L Device:CP1 C?
-U 1 1 5C44521D
-P 7400 5700
-AR Path="/5B50612C/5C44521D" Ref="C?"  Part="1"
-AR Path="/5B5052A9/5C44521D" Ref="C?"  Part="1"
-AR Path="/5FCA9377/5C44521D" Ref="C43"  Part="1"
-F 0 "C43" H 7515 5837 50  0000 L CNN
-F 1 "4.7uF" H 7515 5746 50  0000 L CNN
-F 2 "Capacitor_SMD:C_0402_1005Metric" H 7400 5700 50  0001 C CNN
-F 3 "~" H 7400 5700 50  0001 C CNN
-F 4 "6.3V" H 7515 5655 50  0000 L CNN "Voltage"
-F 5 "0402" H 7515 5564 50  0000 L CNN "SMD size"
-	1    7400 5700
-	1    0    0    -1
-$EndComp
 $Comp
 L Device:CP1 C?
@@
 	8000 5200 8000 5300
 Wire Wire Line
-	8000 5200 7400 5200
-Wire Wire Line
-	7400 5200 7400 5550
-Connection ~ 8000 5200
-Wire Wire Line
-	7400 5850 7400 6200
-Wire Wire Line
-	7400 6200 8000 6200
-Wire Wire Line
 	8000 6200 8000 6100
 Wire Wire Line
@@
 L power:+1V5 #PWR?
 U 1 1 600E13BF
-P 7400 5150
+P 8000 5150
 AR Path="/5FAE186D/600E13BF" Ref="#PWR?"  Part="1"
 AR Path="/5FCA9377/600E13BF" Ref="#PWR0103"  Part="1"
-F 0 "#PWR0103" H 7400 5000 50  0001 C CNN
-F 1 "+1V5" H 7550 5200 50  0000 C CNN
-F 2 "" H 7400 5150 50  0001 C CNN
-F 3 "" H 7400 5150 50  0001 C CNN
-	1    7400 5150
-	1    0    0    -1
-$EndComp
-Wire Wire Line
-	7400 5200 7400 5150
+F 0 "#PWR0103" H 8000 5000 50  0001 C CNN
+F 1 "+1V5" H 8150 5200 50  0000 C CNN
+F 2 "" H 8000 5150 50  0001 C CNN
+F 3 "" H 8000 5150 50  0001 C CNN
+	1    8000 5150
+	1    0    0    -1
+$EndComp
+Wire Wire Line
+	8000 5200 8000 5150
 $Comp
 L power:+1V5 #PWR?
@@
 NoConn ~ 2300 1900
 NoConn ~ 4100 2100
-Wire Bus Line
-	1850 5000 9050 5000
-Wire Bus Line
-	9050 3500 9050 5000
-Wire Bus Line
-	5950 3500 5950 4900
-Wire Bus Line
-	4550 2400 4550 3900
-Wire Bus Line
-	9050 900  9050 2450
-Wire Bus Line
-	1850 2400 1850 5000
 Text Label 8600 1850 0    60   ~ 0
 A7
+Connection ~ 8000 5200
+Wire Bus Line
+	1850 5000 9050 5000
+Wire Bus Line
+	9050 3500 9050 5000
+Wire Bus Line
+	5950 3500 5950 4900
+Wire Bus Line
+	4550 2400 4550 3900
+Wire Bus Line
+	9050 900  9050 2450
+Wire Bus Line
+	1850 2400 1850 5000
 $EndSCHEMATC
