File: _autosave-DDR.sch (KiCad schematic (older format))
At the start: 28 parts, among them U1 IMX6UL_BGA289, U2 DDR3_BGA96

Commit message: Moved some parts to bottom for easier assembly
Parts:
- C46, C47: symbol nano-rescue:CP1 -> Keychain-rescue:CP1-nano-rescue
Changed lines of the file:
@@
 CLK Termination\nClose to DDR3 chip
 $Comp
-L nano-rescue:CP1 C46
+L Keychain-rescue:CP1-nano-rescue C46
 U 1 1 5B4BB0CD
 P 9700 2500
+AR Path="/5B4BB0CD" Ref="C46"  Part="1"
+AR Path="/5FCA9377/5B4BB0CD" Ref="C46"  Part="1"
 F 0 "C46" H 9725 2600 50  0000 L CNN
 F 1 "2.2pF" H 9725 2400 50  0000 L CNN
@@
 $EndComp
 $Comp
-L nano-rescue:CP1 C47
+L Keychain-rescue:CP1-nano-rescue C47
 U 1 1 5B4BB270
 P 9700 2950
+AR Path="/5B4BB270" Ref="C47"  Part="1"
+AR Path="/5FCA9377/5B4BB270" Ref="C47"  Part="1"
 F 0 "C47" H 9725 3050 50  0000 L CNN
 F 1 "2.2pF" H 9725 2850 50  0000 L CNN
